File: reverse-polarity.kicad_pcb (KiCad board)
At the start: 2 copper layers, 37 x 37 mm, 4 parts, among them J1 spring 11m PAD, J2 gnd, J3 105-1102-001, Q1 IRLR9343TRPBF

Commit message: Add files via upload
Parts:
- J2: footprint MountingHole:MountingHole_3.5mm_Pad -> MountingHole:MountingHole_3.2mm_M3_DIN965_Pad
- moved Q1 2.50 mm to (93.5, 43.0)
Routing:
- net /GND: track 96.2 -> 14.4 mm, vias 4 -> 0
- net /+input: track 16.4 -> 9.96 mm
- net /+protected: track 15.8 -> 15.1 mm
- net (no net): vias 0 -> 4
- added copper zone on B.Cu, net (none)
- added copper zone on F.Cu, net (none)
- removed copper zone on B.Cu, net /GND
- removed copper zone on F.Cu, net /GND
Other:
- board size 37 x 37 mm -> 31 x 31 mm
- board text added: "IN"
- board text removed: "BATTERY"
- board text removed: "SPRING"
